File: Nixie/5v_170v_Boost.sch (KiCad schematic (older format))
At the start: 34 parts, among them Q3 MMBTA42, Q4 FDS2672CT, U9 UCC3803

Commit message: Werte angeglichen
Changed lines of the file:
@@
 P 6450 2850
 F 0 "C18" H 6475 2950 50  0000 L CNN
-F 1 "560pF 250v" H 6300 2750 50  0000 L CNN
+F 1 "560pF 250v" H 6250 2750 50  0000 L CNN
 F 2 "Capacitors_SMD:C_0603" H 6488 2700 50  0001 C CNN
 F 3 "https://www.digikey.com/product-detail/en/kemet/C0603C561JAGAC7867/399-14990-1-ND/7382539" H 6450 2850 50  0001 C CNN
@@
 P 5250 2450
 F 0 "C16" H 5275 2550 50  0000 L CNN
-F 1 "100uF 16v" H 5275 2350 50  0000 L CNN
+F 1 "100uF 16v" V 5100 2300 50  0000 L CNN
 F 2 "Capacitors_SMD:C_1210" H 5288 2300 50  0001 C CNN
 F 3 "https://www.digikey.com/product-detail/en/taiyo-yuden/EMK325ABJ107MM-P/587-5426-2-ND/7067011" H 5250 2450 50  0001 C CNN
@@
 P 3600 2450
 F 0 "C12" H 3625 2550 50  0000 L CNN
-F 1 "0.1uF" H 3700 2650 50  0000 L CNN
+F 1 "0.1uF" H 3650 2350 50  0000 L CNN
 F 2 "Capacitors_SMD:C_0805" H 3638 2300 50  0001 C CNN
 F 3 "" H 3600 2450 50  0001 C CNN
@@
 P 3350 2450
 F 0 "C11" H 3375 2550 50  0000 L CNN
-F 1 "100uF 16v" H 3375 2350 50  0000 L CNN
+F 1 "100uF 16v" V 3200 2250 50  0000 L CNN
 F 2 "Capacitors_SMD:C_1210" H 3388 2300 50  0001 C CNN
 F 3 "https://www.digikey.com/product-detail/en/taiyo-yuden/EMK325ABJ107MM-P/587-5426-2-ND/7067011" H 3350 2450 50  0001 C CNN

Commit message: Kleinere Anpassungen
Changed lines of the file:
@@
 L power:GND #PWR039
 U 1 1 58854BC1
-P 4600 4000
-F 0 "#PWR039" H 4600 3750 50  0001 C CNN
-F 1 "GND" H 4600 3850 50  0000 C CNN
-F 2 "" H 4600 4000 50  0000 C CNN
-F 3 "" H 4600 4000 50  0000 C CNN
-	1    4600 4000
+P 4600 3900
+F 0 "#PWR039" H 4600 3650 50  0001 C CNN
+F 1 "GND" H 4600 3750 50  0000 C CNN
+F 2 "" H 4600 3900 50  0000 C CNN
+F 3 "" H 4600 3900 50  0000 C CNN
+	1    4600 3900
 	1    0    0    -1
 $EndComp
@@
 P 4000 4100
 F 0 "R19" V 4080 4100 50  0000 C CNN
-F 1 "0 Ohm" V 3900 4150 50  0000 C CNN
+F 1 "0 Ohm" V 4150 4100 50  0000 C CNN
 F 2 "Resistors_SMD:R_0805" V 3930 4100 50  0001 C CNN
 F 3 "" H 4000 4100 50  0000 C CNN
@@
 P 6700 2400
 F 0 "C19" H 6725 2500 50  0000 L CNN
-F 1 "100pF 250v" H 6700 2200 50  0000 L CNN
+F 1 "100pF 250v" V 6550 2150 50  0000 L CNN
 F 2 "Capacitors_SMD:C_0805" H 6738 2250 50  0001 C CNN
 F 3 "https://www.digikey.com/products/en/capacitors/ceramic-capacitors/60?k=C0805C101JAGAC7800&k=&pkeyword=C0805C101JAGAC7800&pv7=2&quantity=0&ColumnSort=0&page=1&pageSize=25" H 6700 2400 50  0001 C CNN
@@
 $EndComp
 Wire Wire Line
-	4600 4000 4600 3900
-Wire Wire Line
 	4250 2050 4600 2050
