File: Nixie/Nixie.kicad_pcb (KiCad board)
At the start: 2 copper layers, 140 x 80 mm, 45 parts, among them J1 Conn_01x05_Male, J2 Conn_01x02, J3 Barrel_Jack, Q1 BC847, Q2 BC847, SW1 SW_Push, U1 K155ID1, U2 ESP-12E, U3 74HC595, U4 K155ID1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

Commit message: Kleine verschiedene Änderungen
Parts:
- added 3.3V: TestPoint_Pad_D2.5mm, TestPoint:TestPoint_Pad_D2.5mm, F.Cu at (196.0, 90.0)
- added 5V: TestPoint_Pad_D2.5mm, TestPoint:TestPoint_Pad_D2.5mm, F.Cu at (183.0, 79.0)
- added GND: TestPoint_Pad_D2.5mm, TestPoint:TestPoint_Pad_D2.5mm, F.Cu at (207.9, 79.1)
Routing:
- net GND: track 581.5 -> 593.0 mm, vias 10 -> 13
- net +5V: track 307.2 -> 311.5 mm
- net +3.3V: track 208.3 -> 212.3 mm
- added copper zone on F.Cu, net +5V
